Commit message: Added left and right cameras. Need to test validity of positioning.

File: models/cobalt/model.urdf (robot description, URDF)
Before this commit: robot cobalt, 1 links, 0 joints
Links:
- added link left_camera
- added link right_camera
Joints:
- added joint baselink_to_leftcam: type fixed, parent base_link, child left_camera, origin xyz=0.37 0.20 0.04 rpy=-1.57079632679 0 1.57079632679
- added joint baselink_to_rightcam: type fixed, parent base_link, child right_camera, origin xyz=0.37 -0.20 0.04 rpy=-1.57079632679 0 1.57079632679

Commit message: Updated uwsim to add most obstacles.

File: models/cobalt/model.urdf (robot description, URDF)
Before this commit: robot cobalt, 3 links, 2 joints
Links:
- added link bottom_camera
Joints:
- added joint baselink_to_bottomcam: type fixed, parent base_link, child bottom_camera, origin xyz=0.37 -0.20 0.04 rpy=-1.57079632679 0 1.57079632679

Commit message: Added path markers

File: models/cobalt/model.urdf (robot description, URDF)
Before this commit: robot cobalt, 4 links, 3 joints
Joints:
- joint baselink_to_bottomcam: origin xyz=0.37 -0.20 0.04 rpy=-1.57079632679 0 1.57079632679 -> xyz=0 0 0.1 rpy=-1.57079632679 0 1.57079632679
- joint baselink_to_leftcam: origin xyz=0.37 0.20 0.04 rpy=-1.57079632679 0 1.57079632679 -> xyz=0.37 -0.20 0.04 rpy=-1.57079632679 0 1.57079632679
- joint baselink_to_rightcam: origin xyz=0.37 -0.20 0.04 rpy=-1.57079632679 0 1.57079632679 -> xyz=0.37 0.20 0.28 rpy=-1.57079632679 0 1.57079632679
